File: PCB/CrystalBoard.kicad_pcb (KiCad board)
At the start: 2 copper layers, 309.6 x 129.6 mm, 190 parts, among them SW1 SW_Push, SW10 SW_Push, SW11 SW_Push, SW12 SW_Push, SW13 SW_Push, SW17 SW_Push, SW18 SW_Push, SW19 SW_Push, SW2 SW_Push, SW20 SW_Push, SW21 SW_Push, SW22 SW_Push, SW23 SW_Push, SW24 SW_Push, SW25 SW_Push, SW26 SW_Push, SW27 SW_Push, SW28 SW_Push, SW29 SW_Push, SW3 SW_Push, SW30 SW_Push, SW31 SW_Push, SW32 SW_Push, SW33 SW_Push, SW34 SW_Push, SW35 SW_Push, SW36 SW_Push, SW37 SW_Push, SW38 SW_Push, SW39 SW_Push, SW4 SW_Push, SW40 SW_Push, SW41 SW_Push, SW42 SW_Push, SW43 SW_Push, SW44 SW_Push, SW45 SW_Push, SW46 SW_Push, SW47 SW_Push, SW48 SW_Push, SW49 SW_Push, SW5 SW_Push, SW50 SW_Push, SW51 SW_Push, SW52 SW_Push, SW53 SW_Push, SW54 SW_Push, SW55 SW_Push, SW56 SW_Push, SW57 SW_Push, SW58 SW_Push, SW59 SW_Push, SW6 SW_Push, SW60 SW_Push, SW61 SW_Push, SW62 SW_Push, SW63 SW_Push, SW64 SW_Push, SW65 SW_Push, SW66 SW_Push, SW67 SW_Push, SW68 SW_Push, SW69 SW_Push, SW7 SW_Push, SW70 SW_Push, SW71 SW_Push, SW72 SW_Push, SW73 SW_Push, SW74 SW_Push, SW75 SW_Push, SW76 SW_Push, SW77 SW_Push, SW78 SW_Push, SW79 SW_Push, SW8 SW_Push, SW80 SW_Push, SW81 SW_Push, SW82 SW_Push, SW83 SW_Push, SW84 SW_Push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

Commit message: One more Update for re-review
Parts:
- added C1: C, Capacitor_SMD:C_0805_2012Metric_Pad1.18x1.45mm_HandSolder, B.Cu at (284.5, 88.5)
- added C10: C, Capacitor_SMD:C_0805_2012Metric_Pad1.18x1.45mm_HandSolder, B.Cu at (196.5, 183.5)
- added C11: C, Capacitor_SMD:C_0805_2012Metric_Pad1.18x1.45mm_HandSolder, B.Cu at (165.5, 184.0)
- added C12: C, Capacitor_SMD:C_0805_2012Metric_Pad1.18x1.45mm_HandSolder, B.Cu at (133.0, 183.5)
- added C13: C, Capacitor_SMD:C_0805_2012Metric_Pad1.18x1.45mm_HandSolder, B.Cu at (94.0, 184.0)
- added C14: C, Capacitor_SMD:C_0805_2012Metric_Pad1.18x1.45mm_HandSolder, B.Cu at (137.0, 165.0)
- added C15: C, Capacitor_SMD:C_0805_2012Metric_Pad1.18x1.45mm_HandSolder, B.Cu at (156.0, 165.0)
- added C16: C, Capacitor_SMD:C_0805_2012Metric_Pad1.18x1.45mm_HandSolder, B.Cu at (175.0, 165.0)
- added C17: C, Capacitor_SMD:C_0805_2012Metric_Pad1.18x1.45mm_HandSolder, B.Cu at (194.5, 164.5)
- added C18: C, Capacitor_SMD:C_0805_2012Metric_Pad1.18x1.45mm_HandSolder, B.Cu at (213.5, 165.0)
- added C19: C, Capacitor_SMD:C_0805_2012Metric_Pad1.18x1.45mm_HandSolder, B.Cu at (232.5, 164.5)
- added C2: C, Capacitor_SMD:C_0805_2012Metric_Pad1.18x1.45mm_HandSolder, B.Cu at (265.5, 88.5)
- added C20: C, Capacitor_SMD:C_0805_2012Metric_Pad1.18x1.45mm_HandSolder, B.Cu at (251.5, 165.0)
- added C21: C, Capacitor_SMD:C_0805_2012Metric_Pad1.18x1.45mm_HandSolder, B.Cu at (270.5, 165.0)
- added C22: C, Capacitor_SMD:C_0805_2012Metric_Pad1.18x1.45mm_HandSolder, B.Cu at (297.0, 165.0)
- added C23: C, Capacitor_SMD:C_0805_2012Metric_Pad1.18x1.45mm_HandSolder, B.Cu at (323.0, 165.0)
- added C24: C, Capacitor_SMD:C_0805_2012Metric_Pad1.18x1.45mm_HandSolder, B.Cu at (342.0, 164.5)
- added C25: C, Capacitor_SMD:C_0805_2012Metric_Pad1.18x1.45mm_HandSolder, B.Cu at (70.0, 184.0)
- added C26: C, Capacitor_SMD:C_0805_2012Metric_Pad1.18x1.45mm_HandSolder, B.Cu at (46.5, 184.0)
- added C27: C, Capacitor_SMD:C_0805_2012Metric_Pad1.18x1.45mm_HandSolder, B.Cu at (118.0, 165.0)
- added C28: C, Capacitor_SMD:C_0805_2012Metric_Pad1.18x1.45mm_HandSolder, B.Cu at (99.0, 165.0)
- added C29: C, Capacitor_SMD:C_0805_2012Metric_Pad1.18x1.45mm_HandSolder, B.Cu at (68.5, 165.0)
- added C3: C, Capacitor_SMD:C_0805_2012Metric_Pad1.18x1.45mm_HandSolder, B.Cu at (246.8, 88.7)
- added C30: C, Capacitor_SMD:C_0805_2012Metric_Pad1.18x1.45mm_HandSolder, B.Cu at (329.5, 146.0)
- added C31: C, Capacitor_SMD:C_0805_2012Metric_Pad1.18x1.45mm_HandSolder, B.Cu at (298.5, 145.5)
- added C32: C, Capacitor_SMD:C_0805_2012Metric_Pad1.18x1.45mm_HandSolder, B.Cu at (267.5, 145.5)
- added C33: C, Capacitor_SMD:C_0805_2012Metric_Pad1.18x1.45mm_HandSolder, B.Cu at (248.5, 146.0)
- added C34: C, Capacitor_SMD:C_0805_2012Metric_Pad1.18x1.45mm_HandSolder, B.Cu at (229.5, 145.5)
- added C35: C, Capacitor_SMD:C_0805_2012Metric_Pad1.18x1.45mm_HandSolder, B.Cu at (210.5, 145.5)
- added C36: C, Capacitor_SMD:C_0805_2012Metric_Pad1.18x1.45mm_HandSolder, B.Cu at (191.5, 145.5)
- added C37: C, Capacitor_SMD:C_0805_2012Metric_Pad1.18x1.45mm_HandSolder, B.Cu at (172.5, 145.5)
- added C38: C, Capacitor_SMD:C_0805_2012Metric_Pad1.18x1.45mm_HandSolder, B.Cu at (153.5, 145.5)
- added C39: C, Capacitor_SMD:C_0805_2012Metric_Pad1.18x1.45mm_HandSolder, B.Cu at (134.5, 145.5)
- added C4: C, Capacitor_SMD:C_0805_2012Metric_Pad1.18x1.45mm_HandSolder, B.Cu at (329.5, 184.0)
- added C40: C, Capacitor_SMD:C_0805_2012Metric_Pad1.18x1.45mm_HandSolder, B.Cu at (218.0, 126.5)
- added C41: C, Capacitor_SMD:C_0805_2012Metric_Pad1.18x1.45mm_HandSolder, B.Cu at (51.0, 145.5)
- added C42: C, Capacitor_SMD:C_0805_2012Metric_Pad1.18x1.45mm_HandSolder, B.Cu at (77.5, 145.5)
- added C43: C, Capacitor_SMD:C_0805_2012Metric_Pad1.18x1.45mm_HandSolder, B.Cu at (96.5, 145.5)
- added C44: C, Capacitor_SMD:C_0805_2012Metric_Pad1.18x1.45mm_HandSolder, B.Cu at (115.5, 145.5)
- added C45: C, Capacitor_SMD:C_0805_2012Metric_Pad1.18x1.45mm_HandSolder, B.Cu at (61.0, 126.5)
- added C46: C, Capacitor_SMD:C_0805_2012Metric_Pad1.18x1.45mm_HandSolder, B.Cu at (85.0, 126.5)
- added C47: C, Capacitor_SMD:C_0805_2012Metric_Pad1.18x1.45mm_HandSolder, B.Cu at (103.5, 126.5)
- added C48: C, Capacitor_SMD:C_0805_2012Metric_Pad1.18x1.45mm_HandSolder, B.Cu at (122.5, 126.5)
- added C49: C, Capacitor_SMD:C_0805_2012Metric_Pad1.18x1.45mm_HandSolder, B.Cu at (142.0, 126.5)
- added C5: C, Capacitor_SMD:C_0805_2012Metric_Pad1.18x1.45mm_HandSolder, B.Cu at (310.5, 184.0)
- added C50: C, Capacitor_SMD:C_0805_2012Metric_Pad1.18x1.45mm_HandSolder, B.Cu at (161.0, 126.5)
- added C51: C, Capacitor_SMD:C_0805_2012Metric_Pad1.18x1.45mm_HandSolder, B.Cu at (180.0, 126.5)
- added C52: C, Capacitor_SMD:C_0805_2012Metric_Pad1.18x1.45mm_HandSolder, B.Cu at (199.0, 126.5)
- added C53: C, Capacitor_SMD:C_0805_2012Metric_Pad1.18x1.45mm_HandSolder, B.Cu at (237.0, 126.5)
- added C54: C, Capacitor_SMD:C_0805_2012Metric_Pad1.18x1.45mm_HandSolder, B.Cu at (256.0, 126.5)
- added C55: C, Capacitor_SMD:C_0805_2012Metric_Pad1.18x1.45mm_HandSolder, B.Cu at (275.0, 126.5)
- added C56: C, Capacitor_SMD:C_0805_2012Metric_Pad1.18x1.45mm_HandSolder, B.Cu at (294.0, 126.5)
- added C57: C, Capacitor_SMD:C_0805_2012Metric_Pad1.18x1.45mm_HandSolder, B.Cu at (318.0, 126.5)
- added C58: C, Capacitor_SMD:C_0805_2012Metric_Pad1.18x1.45mm_HandSolder, B.Cu at (342.0, 126.5)
- added C59: C, Capacitor_SMD:C_0805_2012Metric_Pad1.18x1.45mm_HandSolder, B.Cu at (329.5, 107.5)
- added C6: C, Capacitor_SMD:C_0805_2012Metric_Pad1.18x1.45mm_HandSolder, B.Cu at (291.5, 184.0)
- added C60: C, Capacitor_SMD:C_0805_2012Metric_Pad1.18x1.45mm_HandSolder, B.Cu at (301.0, 107.5)
- added C61: C, Capacitor_SMD:C_0805_2012Metric_Pad1.18x1.45mm_HandSolder, B.Cu at (272.5, 107.5)
- added C62: C, Capacitor_SMD:C_0805_2012Metric_Pad1.18x1.45mm_HandSolder, B.Cu at (253.5, 107.5)
- added C63: C, Capacitor_SMD:C_0805_2012Metric_Pad1.18x1.45mm_HandSolder, B.Cu at (234.5, 107.5)
- added C64: C, Capacitor_SMD:C_0805_2012Metric_Pad1.18x1.45mm_HandSolder, B.Cu at (215.5, 107.5)
- added C65: C, Capacitor_SMD:C_0805_2012Metric_Pad1.18x1.45mm_HandSolder, B.Cu at (196.5, 107.5)
- added C66: C, Capacitor_SMD:C_0805_2012Metric_Pad1.18x1.45mm_HandSolder, B.Cu at (44.0, 107.5)
- added C67: C, Capacitor_SMD:C_0805_2012Metric_Pad1.18x1.45mm_HandSolder, B.Cu at (63.0, 107.5)
- added C68: C, Capacitor_SMD:C_0805_2012Metric_Pad1.18x1.45mm_HandSolder, B.Cu at (82.0, 107.5)
- added C69: C, Capacitor_SMD:C_0805_2012Metric_Pad1.18x1.45mm_HandSolder, B.Cu at (101.0, 107.5)
- added C7: C, Capacitor_SMD:C_0805_2012Metric_Pad1.18x1.45mm_HandSolder, B.Cu at (272.5, 184.0)
- added C70: C, Capacitor_SMD:C_0805_2012Metric_Pad1.18x1.45mm_HandSolder, B.Cu at (120.0, 107.5)
- added C71: C, Capacitor_SMD:C_0805_2012Metric_Pad1.18x1.45mm_HandSolder, B.Cu at (139.0, 107.5)
- added C72: C, Capacitor_SMD:C_0805_2012Metric_Pad1.18x1.45mm_HandSolder, B.Cu at (158.0, 107.5)
- added C73: C, Capacitor_SMD:C_0805_2012Metric_Pad1.18x1.45mm_HandSolder, B.Cu at (177.5, 107.5)
- added C74: C, Capacitor_SMD:C_0805_2012Metric_Pad1.18x1.45mm_HandSolder, B.Cu at (56.0, 88.5)
- added C75: C, Capacitor_SMD:C_0805_2012Metric_Pad1.18x1.45mm_HandSolder, B.Cu at (75.0, 88.5)
- added C76: C, Capacitor_SMD:C_0805_2012Metric_Pad1.18x1.45mm_HandSolder, B.Cu at (94.5, 88.5)
- added C77: C, Capacitor_SMD:C_0805_2012Metric_Pad1.18x1.45mm_HandSolder, B.Cu at (113.5, 88.5)
- added C78: C, Capacitor_SMD:C_0805_2012Metric_Pad1.18x1.45mm_HandSolder, B.Cu at (132.5, 88.5)
- added C79: C, Capacitor_SMD:C_0805_2012Metric_Pad1.18x1.45mm_HandSolder, B.Cu at (151.5, 88.5)
- added C8: C, Capacitor_SMD:C_0805_2012Metric_Pad1.18x1.45mm_HandSolder, B.Cu at (253.5, 184.0)
- added C80: C, Capacitor_SMD:C_0805_2012Metric_Pad1.18x1.45mm_HandSolder, B.Cu at (170.5, 88.5)
- added C81: C, Capacitor_SMD:C_0805_2012Metric_Pad1.18x1.45mm_HandSolder, B.Cu at (189.5, 88.5)
- added C82: C, Capacitor_SMD:C_0805_2012Metric_Pad1.18x1.45mm_HandSolder, B.Cu at (208.5, 88.5)
- added C83: C, Capacitor_SMD:C_0805_2012Metric_Pad1.18x1.45mm_HandSolder, B.Cu at (227.5, 88.5)
- added C9: C, Capacitor_SMD:C_0805_2012Metric_Pad1.18x1.45mm_HandSolder, B.Cu at (234.5, 184.0)
- added D100: SK6812MINI, Reverse Neopixel:SK6812-MINI-E, B.Cu at (145.3, 107.5)
- added D101: SK6812MINI, Reverse Neopixel:SK6812-MINI-E, B.Cu at (164.3, 107.5)
- added D102: SK6812MINI, Reverse Neopixel:SK6812-MINI-E, B.Cu at (183.4, 107.5)
- added D103: SK6812MINI, Reverse Neopixel:SK6812-MINI-E, B.Cu at (202.4, 107.5)
- added D104: SK6812MINI, Reverse Neopixel:SK6812-MINI-E, B.Cu at (221.5, 107.5)
- added D105: SK6812MINI, Reverse Neopixel:SK6812-MINI-E, B.Cu at (240.5, 107.5)
- added D106: SK6812MINI, Reverse Neopixel:SK6812-MINI-E, B.Cu at (259.6, 107.5)
- added D107: SK6812MINI, Reverse Neopixel:SK6812-MINI-E, B.Cu at (278.6, 107.5)
- added D108: SK6812MINI, Reverse Neopixel:SK6812-MINI-E, B.Cu at (307.2, 107.5)
- added D109: SK6812MINI, Reverse Neopixel:SK6812-MINI-E, B.Cu at (335.8, 107.5)
- added D110: SK6812MINI, Reverse Neopixel:SK6812-MINI-E, B.Cu at (335.8, 126.5)
- added D111: SK6812MINI, Reverse Neopixel:SK6812-MINI-E, B.Cu at (311.9, 126.5)
- added D112: SK6812MINI, Reverse Neopixel:SK6812-MINI-E, B.Cu at (288.1, 126.5)
- added D113: SK6812MINI, Reverse Neopixel:SK6812-MINI-E, B.Cu at (269.1, 126.5)
- added D114: SK6812MINI, Reverse Neopixel:SK6812-MINI-E, B.Cu at (250.0, 126.5)
- added D115: SK6812MINI, Reverse Neopixel:SK6812-MINI-E, B.Cu at (231.0, 126.5)
- added D116: SK6812MINI, Reverse Neopixel:SK6812-MINI-E, B.Cu at (211.9, 126.5)
- added D117: SK6812MINI, Reverse Neopixel:SK6812-MINI-E, B.Cu at (192.9, 126.5)
- added D118: SK6812MINI, Reverse Neopixel:SK6812-MINI-E, B.Cu at (174.0, 126.5)
- added D119: SK6812MINI, Reverse Neopixel:SK6812-MINI-E, B.Cu at (154.8, 126.5)
- added D120: SK6812MINI, Reverse Neopixel:SK6812-MINI-E, B.Cu at (135.7, 126.5)
- added D121: SK6812MINI, Reverse Neopixel:SK6812-MINI-E, B.Cu at (116.7, 126.5)
- added D122: SK6812MINI, Reverse Neopixel:SK6812-MINI-E, B.Cu at (97.6, 126.5)
- added D123: SK6812MINI, Reverse Neopixel:SK6812-MINI-E, B.Cu at (78.6, 126.5)
- added D124: SK6812MINI, Reverse Neopixel:SK6812-MINI-E, B.Cu at (54.8, 126.5)
- added D125: SK6812MINI, Reverse Neopixel:SK6812-MINI-E, B.Cu at (57.1, 145.5)
- added D126: SK6812MINI, Reverse Neopixel:SK6812-MINI-E, B.Cu at (83.3, 145.5)
- added D127: SK6812MINI, Reverse Neopixel:SK6812-MINI-E, B.Cu at (102.4, 145.5)
- added D128: SK6812MINI, Reverse Neopixel:SK6812-MINI-E, B.Cu at (121.4, 145.5)
- added D129: SK6812MINI, Reverse Neopixel:SK6812-MINI-E, B.Cu at (140.5, 145.5)
- added D130: SK6812MINI, Reverse Neopixel:SK6812-MINI-E, B.Cu at (159.5, 145.5)
- added D131: SK6812MINI, Reverse Neopixel:SK6812-MINI-E, B.Cu at (178.6, 145.5)
- added D132: SK6812MINI, Reverse Neopixel:SK6812-MINI-E, B.Cu at (197.6, 145.5)
- added D133: SK6812MINI, Reverse Neopixel:SK6812-MINI-E, B.Cu at (216.7, 145.5)
- added D134: SK6812MINI, Reverse Neopixel:SK6812-MINI-E, B.Cu at (235.7, 145.5)
- added D135: SK6812MINI, Reverse Neopixel:SK6812-MINI-E, B.Cu at (254.8, 145.5)
- added D136: SK6812MINI, Reverse Neopixel:SK6812-MINI-E, B.Cu at (273.8, 145.5)
- added D137: SK6812MINI, Reverse Neopixel:SK6812-MINI-E, B.Cu at (304.8, 145.5)
- added D138: SK6812MINI, Reverse Neopixel:SK6812-MINI-E, B.Cu at (335.8, 145.5)
- added D139: SK6812MINI, Reverse Neopixel:SK6812-MINI-E, B.Cu at (335.8, 164.5)
- added D140: SK6812MINI, Reverse Neopixel:SK6812-MINI-E, B.Cu at (316.7, 164.5)
- added D141: SK6812MINI, Reverse Neopixel:SK6812-MINI-E, B.Cu at (290.5, 164.5)
- added D142: SK6812MINI, Reverse Neopixel:SK6812-MINI-E, B.Cu at (264.3, 164.5)
- added D143: SK6812MINI, Reverse Neopixel:SK6812-MINI-E, B.Cu at (245.3, 164.5)
- added D144: SK6812MINI, Reverse Neopixel:SK6812-MINI-E, B.Cu at (226.2, 164.5)
- added D145: SK6812MINI, Reverse Neopixel:SK6812-MINI-E, B.Cu at (207.2, 164.5)
- added D146: SK6812MINI, Reverse Neopixel:SK6812-MINI-E, B.Cu at (188.1, 164.5)
- added D147: SK6812MINI, Reverse Neopixel:SK6812-MINI-E, B.Cu at (169.1, 164.5)
- added D148: SK6812MINI, Reverse Neopixel:SK6812-MINI-E, B.Cu at (150.0, 164.5)
- added D149: SK6812MINI, Reverse Neopixel:SK6812-MINI-E, B.Cu at (131.0, 164.5)
- added D150: SK6812MINI, Reverse Neopixel:SK6812-MINI-E, B.Cu at (111.9, 164.5)
- added D151: SK6812MINI, Reverse Neopixel:SK6812-MINI-E, B.Cu at (92.9, 164.5)
- added D152: SK6812MINI, Reverse Neopixel:SK6812-MINI-E, B.Cu at (61.9, 164.5)
- added D153: SK6812MINI, Reverse Neopixel:SK6812-MINI-E, B.Cu at (52.4, 183.5)
- added D154: SK6812MINI, Reverse Neopixel:SK6812-MINI-E, B.Cu at (76.2, 183.5)
- added D155: SK6812MINI, Reverse Neopixel:SK6812-MINI-E, B.Cu at (100.0, 183.5)
- added D156: SK6812MINI, Reverse Neopixel:SK6812-MINI-E, B.Cu at (140.0, 183.5)
- added D157: SK6812MINI, Reverse Neopixel:SK6812-MINI-E, B.Cu at (171.4, 183.5)
- added D158: SK6812MINI, Reverse Neopixel:SK6812-MINI-E, B.Cu at (203.5, 183.5)
- added D159: SK6812MINI, Reverse Neopixel:SK6812-MINI-E, B.Cu at (240.5, 183.5)
- added D160: SK6812MINI, Reverse Neopixel:SK6812-MINI-E, B.Cu at (259.6, 183.5)
- added D161: SK6812MINI, Reverse Neopixel:SK6812-MINI-E, B.Cu at (278.6, 183.5)
- added D162: SK6812MINI, Reverse Neopixel:SK6812-MINI-E, B.Cu at (297.7, 183.5)
- added D163: SK6812MINI, Reverse Neopixel:SK6812-MINI-E, B.Cu at (316.7, 183.5)
- added D164: SK6812MINI, Reverse Neopixel:SK6812-MINI-E, B.Cu at (335.8, 183.5)
- added D99: SK6812MINI, Reverse Neopixel:SK6812-MINI-E, B.Cu at (126.2, 107.5)
- D14, D15, D16, D85, D86, D87, D88, D89, D90, D91, D92, D93, D94: footprint LED_SMD:LED_SK6812MINI_PLCC4_3.5x3.5mm_P1.75mm -> Reverse Neopixel:SK6812-MINI-E; moved to B.Cu
- moved D96 65.0 mm to (69.1, 107.5), turned to 180 degrees
- moved D95 51.5 mm to (50.0, 107.5)
- moved D98 45.3 mm to (107.2, 107.5), turned to 180 degrees
- moved D97 41.1 mm to (88.1, 107.5), turned to 180 degrees
- moved D85 21.8 mm to (221.5, 88.5)
- moved D16 21.8 mm to (240.5, 88.5)
- moved D94 21.8 mm to (50.0, 88.5)
- moved D14 21.8 mm to (278.6, 88.5)
- moved D15 21.8 mm to (259.6, 88.5)
- moved D86 21.8 mm to (202.4, 88.5)
- moved D87 21.8 mm to (183.4, 88.5)
- moved D88 21.8 mm to (164.3, 88.5)
- moved D89 21.8 mm to (145.3, 88.5)
- moved D90 21.8 mm to (126.2, 88.5)
- moved D91 21.8 mm to (107.2, 88.5)
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Connections:
- D98 pad 1: unconnected-(D98-DOUT-Pad1) -> Net-(D98-DOUT)
- U1 pad 22: COL16 -> unconnected-(U1-GPIO17-Pad22)_1
- U1 pad 25: ROW3 -> ROW2
- U1 pad 26: ROW2 -> ROW3
Routing:
- net +5V: track 520.4 -> 2694.9 mm
- net GND: track 57.3 -> 222.8 mm, vias 10 -> 148
- net Net-(D94-DOUT): track 114.2 -> 19.7 mm, vias 1 -> 2
- net Net-(D155-DOUT): track 0.00 -> 35.7 mm
- net Net-(D158-DOUT): track 0.00 -> 33.6 mm
- net Net-(D157-DOUT): track 0.00 -> 27.3 mm
- net Net-(D156-DOUT): track 0.00 -> 26.7 mm
- net Net-(D152-DOUT): track 0.00 -> 26.7 mm, vias 0 -> 2
- net Net-(D136-DOUT): track 0.00 -> 26.2 mm
- net Net-(D137-DOUT): track 0.00 -> 26.2 mm
- net Net-(D151-DOUT): track 0.00 -> 26.2 mm, vias 0 -> 2
- net Net-(D108-DOUT): track 0.00 -> 23.8 mm
- net Net-(D107-DOUT): track 0.00 -> 23.8 mm
- net Net-(D95-DOUT): track 37.9 -> 14.3 mm, vias 2 -> 0
- net Net-(D125-DOUT): track 0.00 -> 21.5 mm
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